Commit message: Added camera Modified xacro and gazebo files for a new camera sensor. Added basic image subscriber code. Requires cv2.

File: mrt_ws/src/bot_description/urdf/bot.xacro (robot description, xacro)
@@ -4,4 +4,5 @@
   <xacro:include filename="$(find bot_description)/urdf/bot.gazebo" />
   <xacro:include filename="$(find bot_description)/urdf/macros.xacro" />
+  <xacro:property name="camera_link" value="0.08" /> <!-- Size of square 'camera' box -->
   <link name="link_chassis">
     <!-- pose and inertial -->
@@ -74,4 +75,31 @@
     <child link="sensor_laser"/>
   </joint>
+  <!-- Camera -->
+  <link name="camera_link">
+    <collision>
+      <origin xyz="0 0 0" rpy="0 0 0"/>
+      <geometry>
+        <cylinder radius="0.05" length="0.05"/>
+      </geometry>
+    </collision>
+    <visual>
+      <origin xyz="0 0 0" rpy="0 0 0"/>
+      <geometry>
+        <cylinder radius="0.05" length="0.05"/>
+      </geometry>
+      <material name="green"/>
+    </visual>
+    <inertial>
+      <mass value="1e-5" />
+      <origin xyz="0 0 0" rpy="0 0 0"/>
+      <inertia ixx="1e-6" ixy="0" ixz="0" iyy="1e-6" iyz="0" izz="1e-6" />
+    </inertial>
+  </link>
+  <joint name="camera_joint" type="fixed">
+    <axis xyz="0 1 0" />
+    <origin xyz="0.15 0 0.125" rpy="0 0 0"/>
+    <parent link="link_chassis"/>
+    <child link="camera_link"/>
+  </joint>
   <!-- Create wheel right -->
   <xacro:link_wheel name= "link_right_wheel" />

Commit message: Added arrow+mars Arrow detection script with arrow.world(and launch file) Added mars.world Added IMU sensor

File: mrt_ws/src/bot_description/urdf/bot.xacro (robot description, xacro)
@@ -78,13 +78,13 @@
   <link name="camera_link">
     <collision>
-      <origin xyz="0 0 0" rpy="0 0 0"/>
+      <origin xyz="-0.05 0 0" rpy="0 0 0"/>
       <geometry>
-        <cylinder radius="0.05" length="0.05"/>
+        <cylinder radius="0.005" length="0.005"/>
       </geometry>
     </collision>
     <visual>
-      <origin xyz="0 0 0" rpy="0 0 0"/>
+      <origin xyz="-0.05 0 0" rpy="0 0 0"/>
       <geometry>
-        <cylinder radius="0.05" length="0.05"/>
+        <cylinder radius="0.005" length="0.005"/>
       </geometry>
       <material name="green"/>
@@ -102,4 +102,31 @@
     <child link="camera_link"/>
   </joint>
+  <!-- IMU -->
+  <link name="imu_link">
+    <collision>
+      <origin xyz="0 0 0" rpy="0 0 0"/>
+      <geometry>
+        <cylinder radius="0.05" length="0.05"/>
+      </geometry>
+    </collision>
+    <visual>
+      <origin xyz="0 0 0" rpy="0 0 0"/>
+      <geometry>
+        <cylinder radius="0.05" length="0.05"/>
+      </geometry>
+      <material name="black"/>
+    </visual>
+    <inertial>
+      <mass value="1e-5" />
+      <origin xyz="0 0 0" rpy="0 0 0"/>
+      <inertia ixx="1e-6" ixy="0" ixz="0" iyy="1e-6" iyz="0" izz="1e-6" />
+    </inertial>
+  </link>
+  <joint name="imu_joint" type="fixed">
+    <axis xyz="0 1 0" />
+    <origin xyz="0 0 0.05" rpy="0 0 0"/>
+    <parent link="link_chassis"/>
+    <child link="imu_link"/>
+  </joint>
   <!-- Create wheel right -->
   <xacro:link_wheel name= "link_right_wheel" />
