Commit message: Improved mars world + tuned parameters changed bot.xacro front wheel radius, added a scaled version of bot.xacro for testing Tuned dwa and costmap common params

File: mrt_ws/src/bot_description/urdf/bot2.xacro (robot description, xacro)
@@ -5,15 +5,16 @@
   <xacro:include filename="$(find bot_description)/urdf/macros.xacro" />
   <xacro:property name="camera_link" value="0.08" /> <!-- Size of square 'camera' box -->
+  <xacro:property name="scale" value="2" />
   <link name="link_chassis">
     <!-- pose and inertial -->
-    <pose>0 0 0.1 0 0 0</pose>
+    <pose>0 0 0.25 0 0 0</pose>
     <inertial>
       <mass value="5"/>
-      <origin rpy="0 0 0" xyz="0 0 0.1"/>
+      <origin rpy="0 0 0" xyz="0 0 0.25"/>
       <inertia ixx="0.0395416666667" ixy="0" ixz="0" iyy="0.106208333333" iyz="0" izz="0.106208333333"/>
     </inertial>
     <collision name="collision_chassis">
       <geometry>
-        <box size="0.5 0.3 0.07"/>
+        <box size="1 0.6 0.14"/>
       </geometry>
     </collision>
@@ -21,5 +22,5 @@
       <origin rpy="0 0 0" xyz="0 0 0"/>
       <geometry>
-        <box size="0.5 0.3 0.07"/>
+        <box size="1 0.6 0.14"/>
       </geometry>
       <material name="blue"/>
@@ -27,7 +28,7 @@
     <!-- caster front -->
     <collision name="caster_front_collision">
-      <origin rpy=" 0 0 0" xyz="0.35 0 -0.05"/>
+      <origin rpy=" 0 0 0" xyz="0.7 0 -0.1"/>
       <geometry>
-        <sphere radius="0.06"/>
+        <sphere radius="0.12"/>
       </geometry>
       <surface>
@@ -43,7 +44,7 @@
     </collision>
     <visual name="caster_front_visual">
-      <origin rpy=" 0 0 0" xyz="0.2 0 -0.05"/>
+      <origin rpy=" 0 0 0" xyz="0.4 0 -0.1"/>
       <geometry>
-        <sphere radius="0.06"/>
+        <sphere radius="0.1"/>
       </geometry>
     </visual>
@@ -59,5 +60,5 @@
       <origin xyz="0 0 0" rpy="0 0 0" />
       <geometry>
-        <cylinder radius="0.05" length="0.2"/>
+        <cylinder radius="0.1" length="0.3"/>
       </geometry>
       <material name="white" />
@@ -66,10 +67,11 @@
       <origin xyz="0 0 0" rpy="0 0 0"/>
       <geometry>
-        <cylinder radius="0.05" length="0.2"/>
+        <cylinder radius="0.1" length="0.3"/>
       </geometry>
     </collision>
   </link>
   <joint name="joint_sensor_laser" type="fixed">
-    <origin xyz="0.15 0 0.1" rpy="0 0 0"/>
+    <axis xyz="0 1 0" />
+    <origin xyz="0.3 0 0.15" rpy="0 0 0"/>
     <parent link="link_chassis"/>
     <child link="sensor_laser"/>
@@ -80,5 +82,5 @@
       <origin xyz="0 0 0" rpy="0 0 0"/>
       <geometry>
-        <cylinder radius="0.005" length="0.005"/>
+        <cylinder radius="0.01" length="0.01"/>
       </geometry>
     </collision>
@@ -86,5 +88,5 @@
       <origin xyz="0 0 0" rpy="0 0 0"/>
       <geometry>
-        <cylinder radius="0.005" length="0.005"/>
+        <cylinder radius="0.01" length="0.01"/>
       </geometry>
       <material name="green"/>
@@ -97,6 +99,6 @@
   </link>
   <joint name="camera_joint" type="fixed">
-    <axis xyz="0 1 0" />
-    <origin xyz="0.15 0 0.225" rpy="0 0 0"/>
+    <axis xyz="0 2 0" />
+    <origin xyz="0.3 0 0.25" rpy="0 0 0"/>
     <parent link="link_chassis"/>
     <child link="camera_link"/>
@@ -107,5 +109,5 @@
       <origin xyz="0 0 0" rpy="0 0 0"/>
       <geometry>
-        <cylinder radius="0.05" length="0.05"/>
+        <cylinder radius="0.1" length="0.1"/>
       </geometry>
     </collision>
@@ -113,5 +115,5 @@
       <origin xyz="0 0 0" rpy="0 0 0"/>
       <geometry>
-        <cylinder radius="0.05" length="0.05"/>
+        <cylinder radius="0.1" length="0.1"/>
       </geometry>
       <material name="black"/>
@@ -124,6 +126,6 @@
   </link>
   <joint name="imu_joint" type="fixed">
-    <axis xyz="0 1 0" />
-    <origin xyz="0 0 0.05" rpy="0 0 0"/>
+    <axis xyz="0 2 0" />
+    <origin xyz="0 0 0.1" rpy="0 0 0"/>
     <parent link="link_chassis"/>
     <child link="imu_link"/>
@@ -132,8 +134,8 @@
   <xacro:link_wheel name= "link_right_wheel" />
   <!--   Joint for right wheel  -->
-  <xacro:joint_wheel name="joint_right_wheel"  child="link_right_wheel"  origin_xyz="-0.05 -0.15 0"  />
+  <xacro:joint_wheel name="joint_right_wheel"  child="link_right_wheel"  origin_xyz="-0.1 -0.3 0"  />
   <!-- Left Wheel link -->
   <xacro:link_wheel name= "link_left_wheel" />
   <!--   Joint for right wheel  -->
-  <xacro:joint_wheel name="joint_left_wheel"   child="link_left_wheel"   origin_xyz="-0.05 0.15 0"  />
+  <xacro:joint_wheel name="joint_left_wheel"   child="link_left_wheel"   origin_xyz="-0.1 0.3 0"  />
 </robot>

File: mrt_ws/src/bot_description/urdf/macros.xacro (robot description, xacro)
@@ -27,5 +27,5 @@
         <child link="${child}"/>
         <parent link="link_chassis"/>
-        <axis rpy="0 0 0" xyz="0 1 0"/>
+        <axis rpy="0 0 0" xyz="0 2 0"/>
         <limit effort="10000" velocity="1000"/>
         <joint_properties damping="1.0" friction="1.0"/>
