Commit message: Parameter changes for new model Changed base footprint, link frames and a few parameters

File: mrt_ws/src/bot_description/urdf/rover.urdf (robot description, URDF)
Before this commit: robot rover, 30 links, 29 joints
Joints:
- joint camera_joint: origin xyz=0.56421885520658 -0.526119109974194 0.403679693338444 rpy=0 0 0 -> xyz=-0.06421885520658 -0.526119109974194 0.403679693338444 rpy=0 0 3.1415926
- joint joint_root: origin xyz=-0.27642 0.52612 -0.01368 rpy=0 0 0 -> xyz=0.276421885520658 -0.526119109974194 -0.213679693338444 rpy=0 0 3.1415926
- joint joint_sensor_laser: origin xyz=0.276421885520658 -0.526119109974194 0.413679693338444 rpy=0 0 0 -> xyz=0.276421885520658 -0.526119109974194 0.413679693338444 rpy=0 0 3.1415926

Commit message: Added recovery behaviour, modified arrow detection, added a chess world for camera calibration Changed a few params

File: mrt_ws/src/bot_description/urdf/rover.urdf (robot description, URDF)
Before this commit: robot rover, 30 links, 29 joints
Links:
- added link camera_link_optical
Joints:
- added joint camera_optical_joint: type fixed, parent camera_link, child camera_link_optical, origin xyz=0 0 0 rpy=${-pi/2} 0 ${-pi/2}
