Commit message: urc-ws-imu-added

File: urc_ws/src/bot_description/urdf/bot.xacro (robot description, xacro)
@@ -9,5 +9,5 @@
     <pose>0 0 0.1 0 0 0</pose>
     <inertial>
-      <mass value="5"/>
+      <mass value="20"/>
       <origin rpy="0 0 0" xyz="0 0 0.1"/>
       <inertia ixx="0.0395416666667" ixy="0" ixz="0" iyy="0.106208333333" iyz="0" izz="0.106208333333"/>
@@ -29,5 +29,5 @@
       <origin rpy=" 0 0 0" xyz="0.35 0 -0.05"/>
       <geometry>
-        <sphere radius="0.06"/>
+        <sphere radius="0.05"/>
       </geometry>
       <surface>
@@ -45,5 +45,5 @@
       <origin rpy=" 0 0 0" xyz="0.2 0 -0.05"/>
       <geometry>
-        <sphere radius="0.06"/>
+        <sphere radius="0.05"/>
       </geometry>
     </visual>
